File: MotionBoard Rev C.brd (EAGLE design)
At the start: 99 x 53.3 mm, 110 parts, among them IC1 LPC1769FBD100 or LPC4078FBD10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, IC2 LD1117, IC4 LMV324, Q1 NTGS3441T1G, Q2 12MHz, Q3 25MHz, U1 ARDUINO-FIREPICK+RAMPS, U2 101-00660-68-6, X2 USB-MICRO-B

Commit message: Forgot to update resistor divider values
Signed-off-by: Paul Jones <paul@pauljones.id.au>
Parts:
- R1, R15, R17, R3: value 170k -> 17k
- R16, R18, R2, R6: value 330k -> 33k
Changed lines of the file:
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@@
 <element name="SJ2" library="SparkFun-Passives" package="PAD-JUMPER-2-NC_BY_TRACE_YES_SILK" value="" x="48.5648" y="25.4" rot="MR0"/>
 <element name="SJ3" library="SparkFun-Passives" package="PAD-JUMPER-3-2OF3_NC_BY_TRACE_YES_SILK_FULL_BOX" value="" x="41.8592" y="6.5024" rot="MR90"/>
-<element name="R1" library="Paul" package="0603" value="170k" x="76.6064" y="12.192" smashed="yes" rot="R270">
+<element name="R1" library="Paul" package="0603" value="17k" x="76.6064" y="12.192" smashed="yes" rot="R270">
 <attribute name="NAME" x="77.4192" y="12.9794" size="0.8128" layer="25" font="vector" rot="R270"/>
 <attribute name="VALUE" x="74.9046" y="13.716" size="0.8128" layer="27" font="vector" rot="R270"/>
 </element>
-<element name="R2" library="Paul" package="0603" value="330k" x="80.4672" y="21.9456" rot="R270"/>
+<element name="R2" library="Paul" package="0603" value="33k" x="80.4672" y="21.9456" rot="R270"/>
 <element name="JP1" library="pinhead-2" package="2X04SMD" value="" x="81.6864" y="27.432" rot="R180"/>
-<element name="R3" library="Paul" package="0603" value="170k" x="75.7936" y="16.9672" smashed="yes">
+<element name="R3" library="Paul" package="0603" value="17k" x="75.7936" y="16.9672" smashed="yes">
 <attribute name="NAME" x="74.1426" y="17.3736" size="0.8128" layer="25" font="vector" rot="R180"/>
 <attribute name="VALUE" x="74.2696" y="15.2654" size="0.8128" layer="27" font="vector"/>
 </element>
-<element name="R6" library="Paul" package="0603" value="330k" x="77.8256" y="21.9456" rot="R270"/>
-<element name="R15" library="Paul" package="0603" value="170k" x="85.2424" y="8.8392" smashed="yes">
+<element name="R6" library="Paul" package="0603" value="33k" x="77.8256" y="21.9456" rot="R270"/>
+<element name="R15" library="Paul" package="0603" value="17k" x="85.2424" y="8.8392" smashed="yes">
 <attribute name="NAME" x="83.8962" y="9.3472" size="0.8128" layer="25" font="vector" rot="R180"/>
 <attribute name="VALUE" x="83.7184" y="7.1374" size="0.8128" layer="27" font="vector"/>
 </element>
-<element name="R16" library="Paul" package="0603" value="330k" x="75.3872" y="22.1488" rot="R270"/>
-<element name="R17" library="Paul" package="0603" value="170k" x="86.6648" y="20.4216" smashed="yes" rot="R180">
+<element name="R16" library="Paul" package="0603" value="33k" x="75.3872" y="22.1488" rot="R270"/>
+<element name="R17" library="Paul" package="0603" value="17k" x="86.6648" y="20.4216" smashed="yes" rot="R180">
 <attribute name="NAME" x="87.2998" y="18.5928" size="0.8128" layer="25" font="vector"/>
 <attribute name="VALUE" x="88.1888" y="22.1234" size="0.8128" layer="27" font="vector" rot="R180"/>
 </element>
-<element name="R18" library="Paul" package="0603" value="330k" x="82.9056" y="22.1488" rot="R270"/>
+<element name="R18" library="Paul" package="0603" value="33k" x="82.9056" y="22.1488" rot="R270"/>
 <element name="C21" library="Paul" package="0603" value="100n" x="86.6648" y="21.844" smashed="yes" rot="R180">
 <attribute name="NAME" x="87.6554" y="23.4696" size="0.8128" layer="25" font="vector" rot="R180"/>

Commit message: Update component values
Signed-off-by: Paul Jones <paul@pauljones.id.au>
Parts:
- R52, R7: value 1.5k -> 1k
Routing:
- net TD-: track 18.9 -> 15.3 mm
- net GND: track 65.4 -> 62.9 mm
Changed lines of the file:
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@@
 <attribute name="VALUE" x="30.6832" y="35.6362" size="1.27" layer="27" rot="R270"/>
 </element>
-<element name="R52" library="resistor" package="R0603" value="1.5k" x="34.2392" y="29.1592" smashed="yes" rot="R270">
+<element name="R52" library="resistor" package="R0603" value="1k" x="34.2392" y="29.1592" smashed="yes" rot="R270">
 <attribute name="NAME" x="33.909" y="32.6898" size="0.8128" layer="25" rot="R270"/>
 <attribute name="VALUE" x="32.2072" y="30.0482" size="1.27" layer="27" rot="R270"/>
@@
 <attribute name="VALUE" x="30.48" y="21.6662" size="1.27" layer="27" rot="R90"/>
 </element>
-<element name="R7" library="resistor" package="R0603" value="1.5k" x="10.8204" y="45.72" smashed="yes">
+<element name="R7" library="resistor" package="R0603" value="1k" x="10.8204" y="45.72" smashed="yes">
 <attribute name="NAME" x="11.3538" y="46.8122" size="0.8128" layer="25"/>
 <attribute name="VALUE" x="9.9314" y="43.688" size="1.27" layer="27"/>
@@
 <contactref element="IC7" pad="3"/>
 <contactref element="C44" pad="2"/>
-<contactref element="RJ1" pad="GND"/>
 <contactref element="R61" pad="1"/>
 <contactref element="R50" pad="1"/>
@@
 <wire x1="23.1648" y1="29.2608" x2="22.1488" y2="30.2768" width="0.2032" layer="1"/>
 <wire x1="22.1488" y1="30.2768" x2="21.5138" y2="30.2768" width="0.2032" layer="1"/>
-<wire x1="21.5138" y1="30.2768" x2="19.7612" y2="28.5242" width="0.2032" layer="1"/>
 <via x="59.1312" y="29.2608" extent="1-16" drill="0.381"/>
 <via x="58.42" y="25.6032" extent="1-16" drill="0.381"/>
@@
 <wire x1="21.5392" y1="3.1076" x2="21.5104" y2="3.0788" width="0.2032" layer="1"/>
 <wire x1="19.7104" y1="3.5288" x2="19.7104" y2="4.064" width="0.2032" layer="1"/>
+<contactref element="RJ1" pad="GND"/>
 <wire x1="51.4468" y1="23.0632" x2="49.7468" y2="21.6408" width="0" layer="19" extent="1-1"/>
+<wire x1="21.5138" y1="30.2768" x2="19.7612" y2="28.5242" width="0" layer="19" extent="1-1"/>
 </signal>
 <signal name="3.3V">
@@
 <signal name="TD-">
 <contactref element="IC8" pad="20"/>
-<contactref element="RJ1" pad="TD-"/>
 <contactref element="R55" pad="2"/>
 <contactref element="C55" pad="1"/>
-<wire x1="19.7612" y1="36.1442" x2="20.3454" y2="36.1442" width="0.2032" layer="1"/>
 <wire x1="20.3454" y1="36.1442" x2="20.7264" y2="36.1696" width="0.2032" layer="1"/>
 <wire x1="20.7264" y1="36.1696" x2="23.3308" y2="36.1696" width="0.2032" layer="1"/>
@@
 <via x="21.9456" y="29.0576" extent="1-16" drill="0.3556"/>
 <wire x1="21.9456" y1="29.0576" x2="21.9456" y2="33.9598" width="0.2032" layer="16"/>
-<wire x1="21.9456" y1="33.9598" x2="19.7612" y2="36.1442" width="0.2032" layer="16"/>
+<contactref element="RJ1" pad="TD-"/>
+<wire x1="19.7612" y1="36.1442" x2="20.3454" y2="36.1442" width="0" layer="19" extent="1-1"/>
+<wire x1="21.9456" y1="33.9598" x2="20.7264" y2="36.1696" width="0" layer="19" extent="1-16"/>
 </signal>
 <signal name="RD+">
